File: avionics/hardware/pcb/台灣盃航電倉上層/台灣盃航電倉上層.kicad_sch (KiCad schematic)
At the start: 38 parts, among them J1 SMA, J2 SMA, U1 LIS3MDL, U2 NEO-M9N, U3 E22-900T22S, U4 Connector

Commit message: 對上層PCB的布局進行了一些修改
Parts:
- U4: footprint Connector_PinSocket_2.54mm:PinSocket_2x17_P2.54mm_Vertical -> Connector_PinHeader_1.00mm:PinHeader_2x17_P1.00mm_Vertical
Changed lines of the file:
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@@
 			)
 		)
-		(property "Footprint" "Connector_PinSocket_2.54mm:PinSocket_2x17_P2.54mm_Vertical"
+		(property "Footprint" "Connector_PinHeader_1.00mm:PinHeader_2x17_P1.00mm_Vertical"
 			(at 226.06 85.09 0)
 			(effects
