File: avionics/hardware/pcb/台灣盃航電倉酬載層/台灣盃航電倉酬載層.kicad_sch (KiCad schematic)
At the start: 3 parts, among them U2 MPXV2202DPT1

Commit message: 更新酬載層內容
Parts:
- removed U1: ~, symbol MySymbol:2x16排針母座連接
- removed U2: MPXV2202DPT1, TO_202DPT1_NXP, symbol MPXV2202DPT1:MPXV2202DPT1
- added C1: 220p, Capacitor_SMD:C_0402_1005Metric, symbol Device:C
- added C10, C12, C14, C16, C18, C20, C22, C4, C6, C8: 0.1u, Capacitor_SMD:C_0402_1005Metric, symbol Device:C
- added C11, C19, C24: 100n, Capacitor_SMD:C_0402_1005Metric, symbol Device:C
- added C13, C17, C21, C7: 1u, Capacitor_SMD:C_0402_1005Metric, symbol Device:C
- added C15, C23, C25, C5: 10u, Capacitor_SMD:C_0603_1608Metric, symbol Device:C
- added C2: 4.7u, Capacitor_SMD:C_0603_1608Metric, symbol Device:C
- added C3: 22u, Capacitor_SMD:C_0805_2012Metric, symbol Device:C
- added C9: 2.2u, Capacitor_SMD:C_0603_1608Metric, symbol Device:C
- added D2: MBR0520, Diode_SMD:D_SOD-123, symbol Device:D_Schottky
- added FB1: FerriteBead, Inductor_SMD:L_0603_1608Metric, symbol Device:FerriteBead
- added H1, H2, H3, H4: MountingHole_Pad, MountingHole:MountingHole_2.2mm_M2_DIN965_Pad, symbol Mechanical:MountingHole_Pad
- added L2: 10u, Inductor_SMD:L_1206_3216Metric, symbol Device:L
- added R1: 178K, Resistor_SMD:R_0603_1608Metric, symbol Device:R
- added R2: 24.9K, Resistor_SMD:R_0603_1608Metric, symbol Device:R
- added R3, R4, R5, R6: 2k, Resistor_SMD:R_0603_1608Metric, symbol Device:R
- added R7: 51K, Resistor_SMD:R_0603_1608Metric, symbol Device:R
- added U1, U5, U7, U9: MPXV2202DPT1, MPXV2202DPT1:XDCR_MPXV2202DPT1, symbol MPXV2202DPT1:MPXV2202DPT1
- added U10, U4, U6, U8: INA333xxDGK, Package_SO:VSSOP-8_3x3mm_P0.65mm, symbol Amplifier_Instrumentation:INA333xxDGK
- added U2: LM2733YMF, Package_TO_SOT_SMD:SOT-23-5, symbol Regulator_Switching:LM2733YMF
- U3: value ~ -> Connector; footprint (none) -> Connector_PinHeader_1.00mm:PinHeader_2x17_P1.00mm_Vertical
Connections:
- net GND: now also U3.2 (GND), U3.28 (GND), U3.30 (GND), U3.32 (GND), U3.34 (GND), U3.4 (GND), C10.2, C11.2, C12.2, C13.2, C14.2, C15.2, C16.2, C17.2, C18.2, C19.2, C2.2, C20.2, C21.2, C22.2, C23.2, C24.2, C25.2, C3.2, C4.2, C5.2, C6.2, C7.2, C8.2, C9.2, H1.1, H2.1, H3.1, H4.1, R2.2, U1.1 (GND), U10.4 (V-), U10.5 (Ref), U2.2 (GND), U4.4 (V-), U4.5 (Ref), U5.1 (GND), U6.4 (V-), U6.5 (Ref), U7.1 (GND), U8.4 (V-), U8.5 (Ref), U9.1 (GND)
- net +3V3: now reaches U3.1 (3V3)
- net +3V3: now also U3.29 (3V3), U3.3 (3V3), C10.1, C11.1, C12.1, C15.1, C16.1, C19.1, C20.1, C23.1, U10.7 (V+), U4.7 (V+), U6.7 (V+), U8.7 (V+)
- net PAYLOAD_1: now reaches U3.20 (PAYLOAD_1)
- net PAYLOAD_1: now also U4.6
- net PAYLOAD_2: now reaches U3.22 (PAYLOAD_2)
- net PAYLOAD_2: now also U6.6
- net PAYLOAD_3: now reaches U3.24 (PAYLOAD_3)
- net PAYLOAD_3: now also U8.6
- net PAYLOAD_4: now reaches U3.26 (PAYLOAD_4)
- net PAYLOAD_4: now also U10.6
- net +5V: now reaches U3.31 (5V)
- net +5V: now also C24.1, C25.1, C9.1, L2.1, R7.1, U2.5 (VIN)
- new net: C1.2, C2.1, C3.1, C4.1, D2.1 (K), FB1.1, R1.2
- new net: D2.2 (A), L2.2, U2.1 (SW)
- new net: C1.1, R1.1, R2.1, U2.3 (FB)
- new net: R7.2, U2.4 (EN)
- new net: R5.1, U8.1 (Rg)
- new net: R5.2, U8.8 (Rg)
- new net: R3.1, U4.1 (Rg)
- new net: R3.2, U4.8 (Rg)
- new net: R4.1, U6.1 (Rg)
- new net: R4.2, U6.8 (Rg)
- new net: R6.1, U10.1 (Rg)
- new net: R6.2, U10.8 (Rg)
- new net +10V: C13.1, C14.1, C17.1, C18.1, C21.1, C22.1, C5.1, C6.1, C7.1, C8.1, FB1.2, U1.4 (Vs), U5.4 (Vs), U7.4 (Vs), U9.4 (Vs)
- new net +VOUT_1: U1.2 (+VOUT), U4.3 (+)
- new net +VOUT_2: U5.2 (+VOUT), U6.3 (+)
- new net +VOUT_3: U7.2 (+VOUT), U8.3 (+)
- new net +VOUT_4: U10.3 (+), U9.2 (+VOUT)
- new net -VOUT_1: U1.3 (-VOUT), U4.2 (-)
- new net -VOUT_2: U5.3 (-VOUT), U6.2 (-)
- new net -VOUT_3: U7.3 (-VOUT), U8.2 (-)
- new net -VOUT_4: U10.2 (-), U9.3 (-VOUT)
- no-connect marks 23 -> 20
Other:
- moved on the sheet: U3

Commit message: 完成所有航電板設計
Parts:
- removed C19: 100n, Capacitor_SMD:C_0402_1005Metric, symbol Device:C
- removed C23: 10u, Capacitor_SMD:C_0603_1608Metric, symbol Device:C
- renumbered C16 to C10, C10 to C16
Connections:
- net +3V3: no longer U3.29 (3V3)
- no-connect marks 20 -> 21
