File: avionics/hardware/pcb/台灣盃航電艙第三層_主系統/台灣盃航電艙中層.kicad_pcb (KiCad board)
At the start: 4 copper layers, 80 x 80 mm, 55 parts, among them J2 Micro_SD_Card_Det2, J3 Conn_01x04_Pin, SW1 SW_SPST, U1 STM32F405VGT6, U2 BMI088, U3 BMP390L, U4 Connector, U5 H3LIS331DL, Y1 8MHz

Commit message: 將第一至三層連接器修改成PC104規格，第四層還未進行
Parts:
- removed C23, C26: 10u, Capacitor_SMD:C_0805_2012Metric
- removed C24, C27: 100n, Capacitor_SMD:C_0603_1608Metric
- removed U4: Connector, Connector_PinHeader_1.00mm:PinHeader_2x17_P1.00mm_Vertical
- added C30: 100n, Capacitor_SMD:C_0402_1005Metric, B.Cu at (118.8, 71.9)
- added C31: 10u, Capacitor_SMD:C_0603_1608Metric, B.Cu at (120.0, 72.2)
- added C32: 100n, Capacitor_SMD:C_0402_1005Metric, B.Cu at (174.5, 72.0)
- added C33: 10u, Capacitor_SMD:C_0603_1608Metric, B.Cu at (173.2, 72.2)
- added U11: Connector, Connector_PinHeader_2.54mm:PinHeader_2x20_P2.54mm_Vertical, F.Cu at (122.5, 71.0)
- U3: footprint Bmp390l:XDCR_BMP390L -> BMP390L:XDCR_BMP390L
- Y1: value 8MHz -> 16MHz
Routing:
- net GPS_RESET: track 37.0 -> 59.6 mm, vias 1 -> 3
- net INT_GPS: track 33.4 -> 49.8 mm, vias 1 -> 3
- net SPI2_MOSI: track 73.0 -> 86.7 mm
- net PAYLOAD_1: track 61.4 -> 74.7 mm
- net SPI2_MISO: track 78.0 -> 89.9 mm
- net PAYLOAD_2: track 66.4 -> 77.6 mm, vias 2 -> 3
- net DRDY_MAG: track 27.2 -> 37.8 mm
- net CS_MAG: track 28.2 -> 38.4 mm
- net SPI2_SCK: track 57.0 -> 67.2 mm
- net +3V3: track 46.1 -> 36.3 mm, vias 24 -> 28
- net LORA_M1: track 14.0 -> 23.1 mm
- net INT_MAG: track 27.0 -> 35.3 mm
- net LORA_RESET: track 11.4 -> 19.0 mm
- net LORA_M0: track 12.7 -> 20.3 mm
- net LORA_AUX: track 11.5 -> 18.5 mm
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- added copper zone on B.Cu, net +3V3
- added copper zone on B.Cu, net GND
