File: avionics/hardware/pcb/台灣盃航電艙第四層_供電/台灣盃航電倉下層.kicad_pcb (KiCad board)
At the start: 2 copper layers, 80 x 80 mm, 43 parts, among them J1 XT60, J2 XT60, J4 Pyro1, J5 Pyro2, Q1 NMOS, Q2 NMOS, Q3 NMOS, Q4 NMOS, U3 LM2596S-5, U4 LM2596S-5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

Commit message: Add files via upload
change schematics
Parts:
- U2: footprint Connector_PinHeader_1.00mm:PinHeader_2x02_P1.00mm_Vertical -> Connector_PinHeader_2.54mm:PinHeader_2x02_P2.54mm_Vertical
- moved U2 1.50 mm to (142.5, 72.9)
Routing:
- net +5V_b: track 90.2 -> 91.8 mm
Changed lines of the file:
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@@
 			(outputformat 1)
 			(mirror no)
-			(drillshape 1)
+			(drillshape 0)
 			(scaleselection 1)
-			(outputdirectory "")
+			(outputdirectory "./")
 		)
 	)
@@
 		)
 	)
-	(footprint "Connector_PinHeader_1.00mm:PinHeader_2x02_P1.00mm_Vertical"
+	(footprint "Connector_PinHeader_2.54mm:PinHeader_2x02_P2.54mm_Vertical"
 		(layer "F.Cu")
-		(at 141 72.9 180)
-		(descr "Through hole straight pin header, 2x02, 1.00mm pitch, double rows")
-		(tags "Through hole pin header THT 2x02 1.00mm double row")
+		(at 142.5 72.9 180)
+		(descr "Through hole straight pin header, 2x02, 2.54mm pitch, double rows")
+		(tags "Through hole pin header THT 2x02 2.54mm double row")
 		(property "Reference" "U2"
-			(at 0.5 -1.61 180)
+			(at 1.27 -2.38 0)
 			(layer "F.SilkS")
 			(effects
@@
 		)
 		(property "Value" "~"
-			(at 0.5 2.61 180)
+			(at 1.27 4.92 0)
 			(layer "F.Fab")
 			(effects
@@
 		)
 		(property "Datasheet" ""
-			(at 0 0 180)
+			(at 0 0 0)
 			(layer "F.Fab")
 			(hide yes)
@@
 		)
 		(property "Description" ""
-			(at 0 0 180)
+			(at 0 0 0)
 			(layer "F.Fab")
 			(hide yes)
@@
 		(sheetname "/")
 		(sheetfile "台灣盃航電倉下層.kicad_sch")
+		(zone_connect 2)
 		(attr through_hole)
 		(fp_line
-			(start 1.76 -0.61)
-			(end 1.76 1.61)
+			(start 3.92 -1.38)
+			(end 3.92 3.92)
 			(stroke
 				(width 0.12)
@@
 		)
 		(fp_line
-			(start 1.41003 1.61)
-			(end 1.76 1.61)
+			(start 1.27 1.27)
+			(end 1.27 -1.38)
 			(stroke
 				(width 0.12)
@@
 		)
 		(fp_line
-			(start 1.41003 -0.61)
-			(end 1.76 -0.61)
+			(start 1.27 -1.38)
+			(end 3.92 -1.38)
 			(stroke
 				(width 0.12)
@@
 		)
 		(fp_line
-			(start 0.41003 1.61)
-			(end 0.58997 1.61)
+			(start -1.38 3.92)
+			(end 3.92 3.92)
 			(stroke
 				(width 0.12)
@@
 		)
 		(fp_line
-			(start -0.76 1.61)
-			(end -0.41003 1.61)
+			(start -1.38 1.27)
+			(end 1.27 1.27)
 			(stroke
 				(width 0.12)
@@
 		)
 		(fp_line
-			(start -0.76 0.735)
-			(end -0.685565 0.735)
+			(start -1.38 1.27)
+			(end -1.38 3.92)
 			(stroke
 				(width 0.12)
@@
 		)
 		(fp_line
-			(start -0.76 0.735)
-			(end -0.76 1.61)
+			(start -1.38 0)
+			(end -1.38 -1.38)
 			(stroke
 				(width 0.12)
@@
 		)
 		(fp_line
-			(start -0.76 0)
-			(end -0.76 -0.735)
-			(stroke
-				(width 0.12)
-				(type solid)
-			)
-			(layer "F.SilkS")
-		)
-		(fp_line
-			(start -0.76 -0.735)
-			(end 0 -0.735)
+			(start -1.38 -1.38)
+			(end 0 -1.38)
 			(stroke
 				(width 0.12)
@@
 		)
 		(fp_rect
-			(start -1.15 -1)
-			(end 2.15 2)
+			(start -1.77 -1.77)
+			(end 4.32 4.32)
 			(stroke
 				(width 0.05)
@@
 		)
 		(fp_line
-			(start 1.65 1.5)
-			(end -0.65 1.5)
+			(start 3.81 3.81)
+			(end -1.27 3.81)
 			(stroke
 				(width 0.1)
@@
 		)
 		(fp_line
-			(start 1.65 -0.5)
-			(end 1.65 1.5)
+			(start 3.81 -1.27)
+			(end 3.81 3.81)
 			(stroke
 				(width 0.1)
@@
 		)
 		(fp_line
-			(start -0.075 -0.5)
-			(end 1.65 -0.5)
+			(start 0 -1.27)
+			(end 3.81 -1.27)
 			(stroke
 				(width 0.1)
@@
 		)
 		(fp_line
-			(start -0.65 1.5)
-			(end -0.65 0.075)
+			(start -1.27 3.81)
+			(end -1.27 0)
 			(stroke
 				(width 0.1)
@@
 		)
 		(fp_line
-			(start -0.65 0.075)
-			(end -0.075 -0.5)
+			(start -1.27 0)
+			(end 0 -1.27)
 			(stroke
 				(width 0.1)
@@
 		)
 		(fp_text user "${REFERENCE}"
-			(at 0.5 0.5 270)
+			(at 1.27 1.27 90)
 			(layer "F.Fab")
 			(effects
@@
 		(pad "1" thru_hole rect
 			(at 0 0 180)
-			(size 0.85 0.85)
-			(drill 0.5)
+			(size 1.7 1.7)
+			(drill 1)
 			(layers "*.Cu" "*.Mask")
 			(remove_unused_layers no)
@@
 		)
 		(pad "2" thru_hole circle
-			(at 1 0 180)
-			(size 0.85 0.85)
-			(drill 0.5)
+			(at 2.54 0 180)
+			(size 1.7 1.7)
+			(drill 1)
 			(layers "*.Cu" "*.Mask")
 			(remove_unused_layers no)
@@
 		)
 		(pad "3" thru_hole circle
-			(at 0 1 180)
-			(size 0.85 0.85)
-			(drill 0.5)
+			(at 0 2.54 180)
+			(size 1.7 1.7)
+			(drill 1)
 			(layers "*.Cu" "*.Mask")
 			(remove_unused_layers no)
@@
 		)
 		(pad "4" thru_hole circle
-			(at 1 1 180)
-			(size 0.85 0.85)
-			(drill 0.5)
+			(at 2.54 2.54 180)
+			(size 1.7 1.7)
+			(drill 1)
 			(layers "*.Cu" "*.Mask")
 			(remove_unused_layers no)
@@
 		)
 		(embedded_fonts no)
-		(model "${KICAD9_3DMODEL_DIR}/Connector_PinHeader_1.00mm.3dshapes/PinHeader_2x02_P1.00mm_Vertical.step"
+		(model "${KICAD9_3DMODEL_DIR}/Connector_PinHeader_2.54mm.3dshapes/PinHeader_2x02_P2.54mm_Vertical.step"
 			(offset
 				(xyz 0 0 0)
@@
 	)
 	(segment
-		(start 165.025 104.125)
-		(end 165.025 108.925)
+		(start 164.15 112.45)
+		(end 161.5 112.45)
 		(width 0.2)
 		(layer "F.Cu")
@@
 	)
 	(segment
-		(start 165.025 108.925)
-		(end 161.5 112.45)
+		(start 165.025 104.125)
+		(end 165.025 111.575)
 		(width 0.2)
 		(layer "F.Cu")
@@
 		(layer "F.Cu")
 		(net 5)
+	)
+	(segment
+		(start 165.025 111.575)
+		(end 164.15 112.45)
+		(width 0.2)
+		(layer "F.Cu")
+		(net 5)
