File: avionics/hardware/pcb/台灣盃航電艙第2層_通訊/台灣盃航電倉上層.kicad_pcb (KiCad board)
At the start: 4 copper layers, 80 x 80 mm, 39 parts, among them J1 SMA, J2 SMA, U1 LIS3MDL, U2 NEO-M9N, U3 E22-900T22S, U5 Connector

Commit message: 完成PCB最終設計
Parts:
- J1, J2: footprint Connector_Coaxial:SMA_Amphenol_132134-10_Vertical -> Connector_Coaxial:SMA_Amphenol_132134-11_Vertical
- U3: footprint E22-900T22S:E22-900T22S -> E22-900T22S:PE22-230T22S
- moved U3 14.4 mm to (139.0, 100.5), turned to 0 degrees
- moved C13 3.37 mm to (138.1, 122.0), turned to -10 degrees
- moved R8 3.15 mm to (136.6, 122.6), turned to 80 degrees
- moved C9 3.12 mm to (137.8, 123.9), turned to -10 degrees
- moved C14 2.92 mm to (116.7, 97.0)
- moved C15 2.92 mm to (118.5, 97.2)
- moved J2 2.22 mm to (135.6, 128.6), turned to 80 degrees
- moved C12 1.50 mm to (120.8, 119.0)
- moved R9 1.50 mm to (117.2, 119.0)
Routing:
- net GND: track 26.2 -> 18.1 mm, vias 52 -> 42
- net Net-(J2-In): track 7.29 -> 0.00 mm
- net Net-(U3-ANT): track 5.34 -> 0.33 mm
- net LORA_AUX: track 47.6 -> 49.8 mm
- net LORA_M1: track 47.6 -> 49.3 mm
- net LORA_RX: track 50.3 -> 51.8 mm
- net LORA_TX: track 56.3 -> 55.1 mm
