File: avionics/hardware/pcb/台灣盃航電艙第2層_通訊/台灣盃航電倉上層.kicad_sch (KiCad schematic)
At the start: 38 parts, among them J1 SMA, J2 SMA, U1 LIS3MDL, U2 NEO-M9N, U3 E22-900T22S, U5 Connector

Commit message: 完成PCB最終設計
Parts:
- J1, J2: footprint Connector_Coaxial:SMA_Amphenol_132134-10_Vertical -> Connector_Coaxial:SMA_Amphenol_132134-11_Vertical
- U3: footprint E22-900T22S:E22-900T22S -> E22-900T22S:PE22-230T22S
Changed lines of the file:
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@@
 			)
 		)
-		(property "Footprint" "Connector_Coaxial:SMA_Amphenol_132134-10_Vertical"
+		(property "Footprint" "Connector_Coaxial:SMA_Amphenol_132134-11_Vertical"
 			(at 177.8 54.61 0)
 			(effects
@@
 			)
 		)
-		(property "Footprint" "Connector_Coaxial:SMA_Amphenol_132134-10_Vertical"
+		(property "Footprint" "Connector_Coaxial:SMA_Amphenol_132134-11_Vertical"
 			(at 149.86 73.66 0)
 			(effects
@@
 			)
 		)
-		(property "Footprint" "E22-900T22S:E22-900T22S"
+		(property "Footprint" "E22-900T22S:PE22-230T22S"
 			(at 219.71 27.94 0)
 			(effects
