File: avionics/hardware/pcb/台灣盃航電艙第3層_主系統/台灣盃航電艙中層.kicad_pcb (KiCad board)
At the start: 4 copper layers, 80 x 80 mm, 55 parts, among them J2 Micro_SD_Card_Det2, J3 Conn_01x04_Pin, SW1 SW_SPST, U1 STM32F405VGT6, U11 Connector, U2 BMI088, U3 BMP390L, U5 H3LIS331DL, Y1 16MHz

Commit message: 完成PCB最終設計
Parts:
- U3: value BMP390L -> BMP388
Changed lines of the file:
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@@
 			)
 		)
-		(property "Value" "BMP390L"
+		(property "Value" "BMP388"
 			(at 1.1884 1.5532 0)
 			(layer "F.Fab")
