File: avionics/hardware/pcb/台灣盃航電艙第4層_供電/台灣盃航電倉下層.kicad_pcb (KiCad board)
At the start: 2 copper layers, 80 x 80 mm, 43 parts, among them J1 XT60, J2 XT60, J3 Conn_01x06_Pin, J4 Pyro1, J5 Pyro2, Q1 NMOS, Q2 NMOS, Q3 NMOS, Q4 NMOS, U11 Connector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

Commit message: 更新PCB圖，記得要直接下載PCB檔
Parts:
- moved C6 60.2 mm to (168.4, 124.1), turned to 0 degrees
- moved C8 56.6 mm to (168.4, 122.1), turned to 0 degrees
- moved C10 53.1 mm to (168.4, 120.2), turned to 0 degrees
- moved U6 51.9 mm to (162.1, 121.6), turned to 180 degrees
- moved C12 49.7 mm to (168.4, 118.3), turned to 0 degrees
Routing:
- net +5V_b: track 91.8 -> 37.4 mm
- net +3V3_m: track 31.8 -> 85.4 mm, vias 0 -> 2
- net +BATT_b: track 38.4 -> 68.1 mm
- net +5V_m: track 55.9 -> 68.2 mm, vias 1 -> 2
- net PYRO1: track 57.3 -> 68.6 mm, vias 1 -> 2
- net +BATT_m: track 33.3 -> 43.2 mm
- net +BATT: track 68.3 -> 58.7 mm
- net +3V3_b: track 19.3 -> 22.6 mm
- net GND: track 7.57 -> 4.57 mm, vias 437 -> 4
- net PYRO2: track 50.6 -> 51.5 mm

Commit message: 完成PCB最終設計
Parts:
- added D5: D_M1, Diode_SMD:D_SOD-123, F.Cu at (127.0, 80.0)
- added D6: D_B1, Diode_SMD:D_SOD-123, F.Cu at (172.0, 94.5)
- added D7: D_M2, Diode_SMD:D_SOD-123, B.Cu at (155.5, 83.7)
- added D8: D_B2, Diode_SMD:D_SOD-123, F.Cu at (175.0, 94.5)
- PYRO1: renamed from J4; footprint Connector_JST:JST_XH_B2B-XH-A_1x02_P2.50mm_Vertical -> Connector_JST:JST_XH_S2B-XH-A_1x02_P2.50mm_Horizontal; moved to B.Cu
- PYRO2: renamed from J5; footprint Connector_JST:JST_XH_B2B-XH-A_1x02_P2.50mm_Vertical -> Connector_JST:JST_XH_S2B-XH-A_1x02_P2.50mm_Horizontal
- moved PYRO2 7.67 mm to (138.2, 124.1), turned to 0 degrees
- moved PYRO1 5.63 mm to (134.2, 121.6), turned to 180 degrees
Connections:
- J3 pad 3: +3V3_b -> GND
- J3 pad 5: GND -> B_PYRO1
- J3 pad 6: GND -> B_PYRO2
- R10 pad 2: PYRO1 -> Net-(D5-K)
- R11 pad 1: PYRO1 -> Net-(D5-K)
- R13 pad 2: PYRO2 -> Net-(D7-K)
- R14 pad 1: PYRO2 -> Net-(D7-K)
- U11 pad 20: PYRO1 -> M_PYRO1
- U11 pad 22: PYRO2 -> M_PYRO2
Routing:
- net Net-(D5-K): track 0.00 -> 100.7 mm, vias 0 -> 4
- net PYRO1: track 68.6 -> 0.00 mm, vias 2 -> 0
- net Net-(D7-K): track 0.00 -> 54.2 mm, vias 0 -> 2
- net PYRO2: track 51.5 -> 0.00 mm, vias 1 -> 0
- net M_PYRO1: track 0.00 -> 28.9 mm, vias 0 -> 2
- net M_PYRO2: track 0.00 -> 16.2 mm
- net B_PYRO1: track 0.00 -> 9.32 mm
- net B_PYRO2: track 0.00 -> 6.34 mm
- net Net-(J4-Pin_1): track 11.4 -> 6.21 mm, vias 0 -> 1
- net +BATT: track 58.7 -> 63.2 mm
- net Net-(J5-Pin_1): track 9.82 -> 13.4 mm, vias 0 -> 1
- net +3V3_b: track 22.6 -> 19.9 mm
- net GND: vias 4 -> 381
