File: avionics/hardware/pcb/台灣盃航電艙第5層_次系統/台灣盃航電倉次系統.kicad_pcb (KiCad board)
At the start: 4 copper layers, 80 x 80 mm, 55 parts, among them J1 SH 1.0, J2 Micro_SD_Card, J3 SMA, J4 SMA, J5 Conn_01x04_Pin, J6 Conn_01x06_Pin, SW2 SW_SPST, U1 STM32F103C8Tx, U2 BMP390L, U3 NEO-M9N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

Commit message: 完成PCB最終設計
Parts:
- C19, R12: moved to F.Cu
- J3, J4: footprint Connector_Coaxial:SMA_Amphenol_132134-10_Vertical -> Connector_Coaxial:SMA_Amphenol_132134-11_Vertical
- U6: footprint E22-900T22S:E22-900T22S -> E22-900T22S:PE22-230T22S
- moved D1 44.7 mm to (172.3, 91.5)
- moved R3 44.7 mm to (175.5, 91.5)
- moved U6 14.5 mm to (141.5, 104.3), turned to 90 degrees
- moved SW2 8.35 mm to (116.9, 90.1), turned to 0 degrees
- moved C18 3.93 mm to (121.0, 103.7)
- moved C20 3.93 mm to (123.0, 103.7)
- moved J4 3.93 mm to (114.5, 105.5)
- moved R11 3.93 mm to (122.0, 105.5)
- moved C3 3.83 mm to (119.6, 93.6), turned to 180 degrees
- moved R12 2.83 mm to (127.5, 128.8)
- moved C19 2.56 mm to (127.5, 124.9)
- moved R2 2.39 mm to (123.6, 93.6), turned to 180 degrees
- moved C22 2.00 mm to (144.5, 125.5)
- moved C21 1.54 mm to (144.5, 123.7)
Connections:
- J6 pad 3: +3V3 -> GND
- J6 pad 5: GND -> PYRO_1
- J6 pad 6: GND -> PYRO_2
- U1 pad 19: unconnected-(U1-PB1-Pad19) -> PYRO_1
- U1 pad 20: unconnected-(U1-PB2-Pad20) -> PYRO_2
Routing:
- net PYRO_2: track 0.00 -> 34.5 mm
- net PYRO_1: track 0.00 -> 33.3 mm
- net GND: track 35.6 -> 26.7 mm, vias 67 -> 52
- net LORA_RESET: track 64.6 -> 57.8 mm, vias 1 -> 3
- net Net-(SW2-B): track 26.7 -> 28.7 mm
- net LORA_M0: track 24.0 -> 25.7 mm
- net LORA_M1: track 26.7 -> 28.1 mm
- net LORA_TX: track 22.2 -> 21.2 mm, vias 1 -> 3
- net Net-(U6-ANT): track 5.09 -> 4.16 mm
- net LORA_AUX: track 31.1 -> 31.9 mm, vias 1 -> 3
- net +3V3: track 37.1 -> 37.9 mm, vias 25 -> 24
